File: hardware/BMP280/BMP280_board.sch (EAGLE design)
At the start: 8 parts, among them U1 BMP280, U2 EM406FLAT

Commit message: BMP280
Parts:
- removed C3, C4, C5, C6: 56pF, SparkFun-Capacitors:0.1UF-25V(+80/-20%)(0603)
- added R1: (no value), SparkFun-Passives:RESISTOR0603-RES
- C1: value 0.1uF -> 1.0uF
Connections:
- new net N$1: R1.2, U1.SDO
- net CSB: no longer C3.1
- net GND: no longer C3.2, C4.2, C5.2, C6.2
- net SCK: no longer C5.1
- net SDI: no longer C4.1
- net SDO: now also R1.1; no longer C6.1, U1.SDO
Other:
- note removed: "Protection for overshooting (optional)"
- note removed: "Rozdzielic vdd vddio"
Changed lines of the file:
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@@
 <setting verticaltext="up"/>
 </settings>
-<grid distance="0.1" unitdist="inch" unit="inch" style="lines" multiple="1" display="yes" altdistance="0.01" altunitdist="inch" altunit="inch"/>
+<grid distance="0.1" unitdist="inch" unit="inch" style="lines" multiple="1" display="no" altdistance="0.01" altunitdist="inch" altunit="inch"/>
 <layers>
 <layer number="1" name="Top" color="4" fill="1" visible="no" active="no"/>
@@
 <parts>
 <part name="U1" library="icarus_sensors" deviceset="BMP280" device="_PITCH0.65" value="BMP280"/>
-<part name="GND1" library="SparkFun-Aesthetics" deviceset="GND" device=""/>
 <part name="GND3" library="SparkFun-Aesthetics" deviceset="GND" device=""/>
-<part name="C1" library="SparkFun-Capacitors" deviceset="0.1UF-25V(+80/-20%)(0603)" device="" value="0.1uF"/>
+<part name="C1" library="SparkFun-Capacitors" deviceset="0.1UF-25V(+80/-20%)(0603)" device="" value="1.0uF"/>
 <part name="C2" library="SparkFun-Capacitors" deviceset="0.1UF-25V(+80/-20%)(0603)" device="" value="0.1uF"/>
 <part name="SUPPLY2" library="SparkFun-Aesthetics" deviceset="VCC" device=""/>
 <part name="U2" library="icarus_sensors" deviceset="EM406" device="FLAT"/>
 <part name="SUPPLY1" library="SparkFun-Aesthetics" deviceset="VCC" device=""/>
-<part name="C3" library="SparkFun-Capacitors" deviceset="0.1UF-25V(+80/-20%)(0603)" device="" value="56pF"/>
-<part name="C4" library="SparkFun-Capacitors" deviceset="0.1UF-25V(+80/-20%)(0603)" device="" value="56pF"/>
-<part name="C5" library="SparkFun-Capacitors" deviceset="0.1UF-25V(+80/-20%)(0603)" device="" value="56pF"/>
-<part name="C6" library="SparkFun-Capacitors" deviceset="0.1UF-25V(+80/-20%)(0603)" device="" value="56pF"/>
 <part name="GND2" library="SparkFun-Aesthetics" deviceset="GND" device=""/>
-<part name="GND5" library="SparkFun-Aesthetics" deviceset="GND" device=""/>
-<part name="GND6" library="SparkFun-Aesthetics" deviceset="GND" device=""/>
-<part name="GND7" library="SparkFun-Aesthetics" deviceset="GND" device=""/>
 <part name="GND8" library="SparkFun-Aesthetics" deviceset="GND" device=""/>
+<part name="R1" library="SparkFun-Passives" deviceset="RESISTOR" device="0603-RES"/>
 </parts>
 <sheets>
 <sheet>
 <plain>
-<wire x1="-33.02" y1="-15.24" x2="48.26" y2="-15.24" width="0.1524" layer="97" style="longdash"/>
-<wire x1="48.26" y1="-15.24" x2="48.26" y2="-38.1" width="0.1524" layer="97" style="longdash"/>
-<wire x1="48.26" y1="-38.1" x2="-33.02" y2="-38.1" width="0.1524" layer="97" style="longdash"/>
-<wire x1="-33.02" y1="-38.1" x2="-33.02" y2="-15.24" width="0.1524" layer="97" style="longdash"/>
-<text x="-32.258" y="-37.338" size="1.778" layer="97">Protection for overshooting (optional)</text>
-<text x="-35.56" y="38.1" size="1.778" layer="97">Rozdzielic vdd vddio</text>
 </plain>
 <instances>
 <instance part="U1" gate="G$1" x="0" y="0"/>
-<instance part="GND1" gate="1" x="30.48" y="-30.48"/>
-<instance part="GND3" gate="1" x="68.58" y="-30.48"/>
+<instance part="GND3" gate="1" x="68.58" y="-10.16"/>
 <instance part="C1" gate="G$1" x="-27.94" y="12.7" rot="R270"/>
 <instance part="C2" gate="G$1" x="-27.94" y="22.86" rot="R270"/>
@@
 <instance part="U2" gate="G$1" x="88.9" y="5.08"/>
 <instance part="SUPPLY1" gate="G$1" x="68.58" y="27.94"/>
-<instance part="C3" gate="G$1" x="38.1" y="-22.86"/>
-<instance part="C4" gate="G$1" x="30.48" y="-22.86"/>
-<instance part="C5" gate="G$1" x="22.86" y="-22.86"/>
-<instance part="C6" gate="G$1" x="-20.32" y="-22.86"/>
 <instance part="GND2" gate="1" x="-33.02" y="30.48" rot="R180"/>
-<instance part="GND5" gate="1" x="-20.32" y="-30.48"/>
-<instance part="GND6" gate="1" x="22.86" y="-30.48"/>
-<instance part="GND7" gate="1" x="38.1" y="-30.48"/>
 <instance part="GND8" gate="1" x="22.86" y="30.48" rot="R180"/>
+<instance part="R1" gate="G$1" x="-22.86" y="-7.62"/>
 </instances>
 <busses>
@@
 <pinref part="GND3" gate="1" pin="GND"/>
 <wire x1="76.2" y1="-2.54" x2="68.58" y2="-2.54" width="0.1524" layer="91"/>
-<wire x1="68.58" y1="-2.54" x2="68.58" y2="-27.94" width="0.1524" layer="91"/>
+<wire x1="68.58" y1="-2.54" x2="68.58" y2="-7.62" width="0.1524" layer="91"/>
 </segment>
 <segment>
@@
 <junction x="-33.02" y="22.86"/>
 </segment>
-<segment>
-<pinref part="C6" gate="G$1" pin="2"/>
-<wire x1="-20.32" y1="-25.4" x2="-20.32" y2="-27.94" width="0.1524" layer="91"/>
-<pinref part="GND5" gate="1" pin="GND"/>
-</segment>
-<segment>
-<pinref part="C5" gate="G$1" pin="2"/>
-<wire x1="22.86" y1="-25.4" x2="22.86" y2="-27.94" width="0.1524" layer="91"/>
-<pinref part="GND6" gate="1" pin="GND"/>
-</segment>
-<segment>
-<pinref part="C3" gate="G$1" pin="2"/>
-<wire x1="38.1" y1="-25.4" x2="38.1" y2="-27.94" width="0.1524" layer="91"/>
-<pinref part="GND7" gate="1" pin="GND"/>
-</segment>
-<segment>
-<pinref part="C4" gate="G$1" pin="2"/>
-<wire x1="30.48" y1="-25.4" x2="30.48" y2="-27.94" width="0.1524" layer="91"/>
-<pinref part="GND1" gate="1" pin="GND"/>
-</segment>
 </net>
 <net name="CSB" class="0">
@@
 <pinref part="U1" gate="G$1" pin="CSB"/>
 <label x="43.18" y="2.54" size="1.778" layer="95"/>
-<pinref part="C3" gate="G$1" pin="1"/>
-<wire x1="17.78" y1="2.54" x2="38.1" y2="2.54" width="0.1524" layer="91"/>
-<wire x1="38.1" y1="2.54" x2="38.1" y2="-17.78" width="0.1524" layer="91"/>
-<wire x1="38.1" y1="2.54" x2="48.26" y2="2.54" width="0.1524" layer="91"/>
-<junction x="38.1" y="2.54"/>
+<wire x1="17.78" y1="2.54" x2="48.26" y2="2.54" width="0.1524" layer="91"/>
 </segment>
 <segment>
@@
 <pinref part="U1" gate="G$1" pin="SCK"/>
 <label x="43.18" y="-7.62" size="1.778" layer="95"/>
-<pinref part="C5" gate="G$1" pin="1"/>
-<wire x1="17.78" y1="-7.62" x2="22.86" y2="-7.62" width="0.1524" layer="91"/>
-<wire x1="22.86" y1="-7.62" x2="22.86" y2="-17.78" width="0.1524" layer="91"/>
-<wire x1="22.86" y1="-7.62" x2="48.26" y2="-7.62" width="0.1524" layer="91"/>
-<junction x="22.86" y="-7.62"/>
+<wire x1="17.78" y1="-7.62" x2="48.26" y2="-7.62" width="0.1524" layer="91"/>
 </segment>
 <segment>
@@
 <net name="SDO" class="0">
 <segment>
-<pinref part="U1" gate="G$1" pin="SDO"/>
-<wire x1="-17.78" y1="-7.62" x2="-20.32" y2="-7.62" width="0.1524" layer="91"/>
-<label x="-33.02" y="-7.62" size="1.778" layer="95"/>
-<pinref part="C6" gate="G$1" pin="1"/>
-<wire x1="-20.32" y1="-7.62" x2="-20.32" y2="-17.78" width="0.1524" layer="91"/>
-<wire x1="-20.32" y1="-7.62" x2="-33.02" y2="-7.62" width="0.1524" layer="91"/>
-<junction x="-20.32" y="-7.62"/>
-</segment>
-<segment>
 <pinref part="U2" gate="G$1" pin="SDO"/>
 <wire x1="76.2" y1="7.62" x2="68.58" y2="7.62" width="0.1524" layer="91"/>
 <label x="68.58" y="7.62" size="1.778" layer="95"/>
 </segment>
+<segment>
+<pinref part="R1" gate="G$1" pin="1"/>
+<wire x1="-27.94" y1="-7.62" x2="-33.02" y2="-7.62" width="0.1524" layer="91"/>
+<label x="-33.02" y="-7.62" size="1.778" layer="95"/>
+</segment>
 </net>
 <net name="SDI" class="0">
@@
 <pinref part="U1" gate="G$1" pin="SDI"/>
 <label x="43.18" y="-2.54" size="1.778" layer="95"/>
-<pinref part="C4" gate="G$1" pin="1"/>
-<wire x1="17.78" y1="-2.54" x2="30.48" y2="-2.54" width="0.1524" layer="91"/>
-<wire x1="30.48" y1="-2.54" x2="30.48" y2="-17.78" width="0.1524" layer="91"/>
-<wire x1="30.48" y1="-2.54" x2="48.26" y2="-2.54" width="0.1524" layer="91"/>
-<junction x="30.48" y="-2.54"/>
+<wire x1="17.78" y1="-2.54" x2="48.26" y2="-2.54" width="0.1524" layer="91"/>
 </segment>
 <segment>
@@
 </segment>
 </net>
+<net name="N$1" class="0">
+<segment>
+<pinref part="U1" gate="G$1" pin="SDO"/>
+<pinref part="R1" gate="G$1" pin="2"/>
+</segment>
+</net>
