File: hardware/shield/new_9DOF.brd (EAGLE design)
At the start: 23.9 x 32.2 mm, 37 parts, among them IC3 FM25-DFN, T2 BC846, U1 EM406FLAT, U2 EM406FLAT, U4 EM406FLAT, U5 ADXL362, U6 W25Q16BVZP, U7 MPU-9250, X1 NRF51822-RIGHT

Commit message: shield
Parts:
- moved C14 52.2 mm to (11.6, 29.9), flipped to the bottom, turned to 270 degrees
- moved C13 48.7 mm to (9.14, 29.8), flipped to the bottom, turned to 270 degrees
- moved C11 42.4 mm to (6.45, 29.9), flipped to the bottom, turned to 270 degrees
- moved C12 20.8 mm to (12.0, 1.94), flipped to the bottom, turned to 270 degrees
- moved C10 14.0 mm to (8.75, 1.99), flipped to the bottom, turned to 270 degrees
- moved C4 13.2 mm to (21.8, 21.1)
- moved C3 11.7 mm to (16.4, 29.8)
- moved C9 10.4 mm to (6.72, 1.99), flipped to the bottom, turned to 90 degrees
- moved U$4 8.19 mm to (7.20, 17.2), flipped to the bottom, turned to 270 degrees
- moved R9 5.09 mm to (10.4, 5.75)
- moved R7 4.45 mm to (6.97, 5.67)
- moved R2 4.10 mm to (10.6, 17.2), turned to 180 degrees
- moved C1 3.61 mm to (14.0, 29.9), turned to 270 degrees
- moved U5 2.97 mm to (3.97, 25.2)
- moved C7 2.72 mm to (8.07, 10.0)
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Connections:
- net ADXL_CS: now also U$1.4; no longer U$1.10
- net ADXL_DATA: now also U$1.2; no longer U$1.8
- net ADXL_FSYNC: now also U$1.3; no longer U$1.7
- net BAR1_CS: now also U$1.6; no longer U$1.2
- net N$3: now also U$1.7; no longer U$1.3
- net N$4: now also U$1.8; no longer U$1.4
- net SWITCH: now also X1.8; no longer X1.6
Routing:
- net VCCIO: track 40.4 -> 2.88 mm, vias 4 -> 0
- net GND: track 123.8 -> 160.4 mm, vias 10 -> 4
- net SCK1: track 39.1 -> 55.8 mm, vias 3 -> 4
- net SDO2: track 23.7 -> 35.0 mm
- net SDI2: track 11.2 -> 22.2 mm, vias 0 -> 3
- net VIN: track 4.77 -> 15.1 mm, vias 0 -> 1
- net N$1: track 20.1 -> 13.6 mm
- net SCK2: track 15.3 -> 20.7 mm, vias 0 -> 2
- net N$8: track 3.11 -> 8.41 mm
- net SDI1: track 47.8 -> 42.5 mm, vias 4 -> 6
- net VCC: track 113.5 -> 118.7 mm, vias 12 -> 13
- net BAR3_CS: track 26.3 -> 22.0 mm, vias 0 -> 1
- net N$5: track 8.31 -> 4.13 mm
- net FLASH_HOLD: track 10.3 -> 6.21 mm, vias 1 -> 0
- net MPU_CS: track 9.00 -> 13.0 mm, vias 0 -> 1
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