File: hardware/shield/new_9DOF.sch (EAGLE design)
At the start: 37 parts, among them IC3 FM25-DFN, T2 BC846, U1 EM406FLAT, U2 EM406FLAT, U4 EM406FLAT, U5 ADXL362, U6 W25Q16BVZP, U7 MPU-9250, X1 NRF51822-RIGHT

Commit message: shield
Connections:
- net ADXL_CS: now also U$1P0.23.S; no longer U$1P0.29.S
- net ADXL_DATA: now also U$1P0.21.S; no longer U$1P0.27.S
- net ADXL_FSYNC: now also U$1P0.22.S; no longer U$1P0.26.S
- net BAR1_CS: now also U$1P0.25.S; no longer U$1P0.21.S
- net N$3: now also U$1P0.26.S; no longer U$1P0.22.S
- net N$4: now also U$1P0.27.S; no longer U$1P0.23.S
- net SWITCH: now also X1P0.16.S; no longer X1SWD.S
Other:
- moved on the sheet: R2, R4
Changed lines of the file:
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@@
 <instance part="T2" gate="G$1" x="137.16" y="17.78" rot="R180"/>
 <instance part="R1" gate="G$1" x="121.92" y="15.24"/>
-<instance part="R2" gate="G$1" x="45.72" y="45.72" rot="R180"/>
-<instance part="R4" gate="G$1" x="-2.54" y="45.72" rot="R180"/>
+<instance part="R2" gate="G$1" x="45.72" y="40.64" rot="R180"/>
+<instance part="R4" gate="G$1" x="-10.16" y="40.64" rot="R180"/>
 <instance part="U2" gate="G$1" x="228.6" y="93.98"/>
 <instance part="U$4" gate="G$1" x="53.34" y="83.82" rot="MR0"/>
@@
 </segment>
 <segment>
-<pinref part="U$1" gate="P0.21" pin="S"/>
-<wire x1="38.1" y1="48.26" x2="48.26" y2="48.26" width="0.1524" layer="91"/>
-<label x="40.64" y="48.26" size="1.778" layer="95"/>
+<pinref part="U$1" gate="P0.25" pin="S"/>
+<wire x1="38.1" y1="43.18" x2="48.26" y2="43.18" width="0.1524" layer="91"/>
+<label x="40.64" y="43.18" size="1.778" layer="95"/>
 </segment>
 </net>
@@
 </segment>
 <segment>
-<pinref part="U$1" gate="P0.29" pin="S"/>
-<wire x1="38.1" y1="38.1" x2="48.26" y2="38.1" width="0.1524" layer="91"/>
-<label x="40.64" y="38.1" size="1.778" layer="95"/>
+<pinref part="U$1" gate="P0.23" pin="S"/>
+<wire x1="38.1" y1="45.72" x2="48.26" y2="45.72" width="0.1524" layer="91"/>
+<label x="40.64" y="45.72" size="1.778" layer="95"/>
 </segment>
 </net>
@@
 </segment>
 <segment>
-<pinref part="U$1" gate="P0.27" pin="S"/>
-<wire x1="38.1" y1="40.64" x2="48.26" y2="40.64" width="0.1524" layer="91"/>
-<label x="40.64" y="40.64" size="1.778" layer="95"/>
+<pinref part="U$1" gate="P0.21" pin="S"/>
+<wire x1="38.1" y1="48.26" x2="48.26" y2="48.26" width="0.1524" layer="91"/>
+<label x="40.64" y="48.26" size="1.778" layer="95"/>
 </segment>
 </net>
@@
 </segment>
 <segment>
-<pinref part="U$1" gate="P0.26" pin="S"/>
-<wire x1="5.08" y1="40.64" x2="-15.24" y2="40.64" width="0.1524" layer="91"/>
-<label x="-15.24" y="40.64" size="1.778" layer="95"/>
+<pinref part="U$1" gate="P0.22" pin="S"/>
+<wire x1="5.08" y1="45.72" x2="-2.54" y2="45.72" width="0.1524" layer="91"/>
+<label x="-7.62" y="45.72" size="1.778" layer="95"/>
 </segment>
 </net>
@@
 </segment>
 <segment>
-<pinref part="X1" gate="SWD" pin="S"/>
-<wire x1="193.04" y1="43.18" x2="203.2" y2="43.18" width="0.1524" layer="91"/>
-<label x="195.58" y="43.18" size="1.778" layer="95"/>
+<pinref part="X1" gate="P0.16" pin="S"/>
+<wire x1="193.04" y1="40.64" x2="203.2" y2="40.64" width="0.1524" layer="91"/>
+<label x="195.58" y="40.64" size="1.778" layer="95"/>
 </segment>
 </net>
@@
 <pinref part="R2" gate="G$1" pin="1"/>
 <label x="73.66" y="45.72" size="1.778" layer="95"/>
-<wire x1="50.8" y1="45.72" x2="66.04" y2="45.72" width="0.1524" layer="91"/>
+<wire x1="50.8" y1="40.64" x2="66.04" y2="43.18" width="0.1524" layer="91"/>
 <pinref part="C11" gate="G$1" pin="2"/>
-<wire x1="66.04" y1="45.72" x2="78.74" y2="45.72" width="0.1524" layer="91"/>
-<wire x1="66.04" y1="45.72" x2="66.04" y2="48.26" width="0.1524" layer="91"/>
-<junction x="66.04" y="45.72"/>
+<wire x1="66.04" y1="43.18" x2="78.74" y2="43.18" width="0.1524" layer="91"/>
+<wire x1="66.04" y1="43.18" x2="66.04" y2="48.26" width="0.1524" layer="91"/>
+<junction x="66.04" y="43.18"/>
 </segment>
 </net>
@@
 <segment>
 <pinref part="R4" gate="G$1" pin="2"/>
-<label x="-33.02" y="45.72" size="1.778" layer="95"/>
+<label x="-33.02" y="40.64" size="1.778" layer="95"/>
 <pinref part="C14" gate="G$1" pin="2"/>
-<wire x1="-7.62" y1="45.72" x2="-25.4" y2="45.72" width="0.1524" layer="91"/>
-<wire x1="-25.4" y1="45.72" x2="-25.4" y2="53.34" width="0.1524" layer="91"/>
-<wire x1="-25.4" y1="45.72" x2="-33.02" y2="45.72" width="0.1524" layer="91"/>
-<junction x="-25.4" y="45.72"/>
+<wire x1="-15.24" y1="40.64" x2="-25.4" y2="40.64" width="0.1524" layer="91"/>
+<wire x1="-25.4" y1="40.64" x2="-25.4" y2="53.34" width="0.1524" layer="91"/>
+<wire x1="-25.4" y1="40.64" x2="-33.02" y2="40.64" width="0.1524" layer="91"/>
+<junction x="-25.4" y="40.64"/>
 </segment>
 </net>
@@
 <net name="SDO2" class="0">
 <segment>
-<pinref part="U6" gate="G$1" pin="DO"/>
-<wire x1="60.96" y1="142.24" x2="48.26" y2="142.24" width="0.1524" layer="91"/>
-<label x="48.26" y="142.24" size="1.778" layer="95"/>
-</segment>
-<segment>
 <pinref part="IC3" gate="G$1" pin="DO"/>
 <wire x1="30.48" y1="139.7" x2="38.1" y2="139.7" width="0.1524" layer="91"/>
@@
 <wire x1="-25.4" y1="27.94" x2="-33.02" y2="27.94" width="0.1524" layer="91"/>
 </segment>
+<segment>
+<pinref part="U6" gate="G$1" pin="DO"/>
+<wire x1="60.96" y1="142.24" x2="48.26" y2="142.24" width="0.1524" layer="91"/>
+<label x="48.26" y="142.24" size="1.778" layer="95"/>
+</segment>
 </net>
 <net name="SCK2" class="0">
@@
 </segment>
 </net>
-<net name="N$3" class="0">
-<segment>
-<pinref part="R4" gate="G$1" pin="1"/>
-<pinref part="U$1" gate="P0.22" pin="S"/>
-<wire x1="2.54" y1="45.72" x2="5.08" y2="45.72" width="0.1524" layer="91"/>
-</segment>
-</net>
-<net name="N$4" class="0">
-<segment>
-<pinref part="U$1" gate="P0.23" pin="S"/>
-<pinref part="R2" gate="G$1" pin="2"/>
-<wire x1="38.1" y1="45.72" x2="40.64" y2="45.72" width="0.1524" layer="91"/>
-</segment>
-</net>
 <net name="N$5" class="0">
 <segment>
@@
 </segment>
 </net>
+<net name="N$3" class="0">
+<segment>
+<pinref part="R4" gate="G$1" pin="1"/>
+<pinref part="U$1" gate="P0.26" pin="S"/>
+<wire x1="-5.08" y1="40.64" x2="5.08" y2="40.64" width="0.1524" layer="91"/>
+</segment>
+</net>
+<net name="N$4" class="0">
+<segment>
+<pinref part="R2" gate="G$1" pin="2"/>
+<pinref part="U$1" gate="P0.27" pin="S"/>
+<wire x1="40.64" y1="40.64" x2="38.1" y2="40.64" width="0.1524" layer="91"/>
+</segment>
+</net>
